File: HSLinkIsolate.kicad_pcb (KiCad board)
At the start: 2 copper layers, 65 x 40 mm, 62 parts, among them J101 USB_B, J102 ISP, J103 IDC, Q101 AO3400A, SW101 BOOT, U101 HPM5301IEG1, U102 USBLC6-2SC6, U103 ISO7741, U104 ISO7741, U105 SN74LVC1G125DBV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

Commit message: modify pcb
Parts:
- moved C110 0.10 mm to (201.3, 106.3)
Routing:
- net VDD_SOC: track 94.9 -> 87.6 mm
- net /SW: track 4.83 -> 0.00 mm
- net GND1: vias 10 -> 16
- net GND: vias 16 -> 59
- added copper zone on F.Cu, net /SW
- added copper zone on F.Cu, net VDD_SOC
Other:
- board text added: "JLCJLCJLCJLC"
